File: Elektronika_K001_DON_Keyboard/Elektronika_K001_DON_Keyboard.kicad_pcb (KiCad board)
At the start: 2 copper layers, 300 x 130 mm, 74 parts, among them J1 ROWS, J2 COLS, SW1 СБР, SW10 1, SW11 C, SW12 Y, SW13 ⎴, SW14 ↖, SW15 NEW, SW16 2, SW17 U, SW18 W, SW19 S, SW2 НР, SW20 ↑, SW21 LOAD, SW22 3, SW23 K, SW24 A, SW25 M, SW26 ↓, SW27 SAVE, SW28 4, SW29 E, SW3 FUNC, SW30 P, SW31 I, SW32 RUN, SW33 5, SW34 N, SW35 R, SW36 T, SW37 STOP, SW38 6, SW39 G, SW4 +, SW40 O, SW41 X, SW42 SPACE, SW43 CONT, SW44 7, SW45 [, SW46 L, SW47 B, SW48 ←, SW49 EDIT, SW5 J, SW50 8, SW51 ], SW52 D, SW53 @, SW54 ПВ, SW55 ◼, SW56 9, SW57 Z, SW58 V, SW59 <, SW6 F, SW60 →, SW61 ◻, SW62 0, SW63 H, SW64 \, SW65 ?, SW66 ПС, SW67 ⎅, SW68 =, SW69 *, SW7 Q, SW70 >, SW71 ЗБ, SW72 ВК, SW8 НР ФИКС, SW9 HELP

Commit message: Finalised design for testing
Parts:
- moved J2 165.1 mm to (352.8, 120.5), turned to 0 degrees
- moved J1 133.9 mm to (69.1, 128.4), turned to 0 degrees
Routing:
- net /ROW_B: track 478.7 -> 263.7 mm
- net /ROW_C: track 461.5 -> 248.0 mm
- net /ROW_D: track 442.7 -> 245.9 mm
- net /COL_2: track 216.2 -> 403.1 mm
- net /COL_3: track 200.6 -> 384.6 mm
- net /ROW_E: track 424.4 -> 249.4 mm
- net /COL_4: track 183.7 -> 344.7 mm
- net /COL_5: track 167.1 -> 323.1 mm
- net /ROW_F: track 405.1 -> 261.0 mm
- net /COL_6: track 143.7 -> 280.2 mm
- net /COL_7: track 142.1 -> 260.2 mm
- net /COL_8: track 147.3 -> 262.0 mm
- net /COL_9: track 121.2 -> 230.6 mm
- net /COL_10: track 133.5 -> 207.4 mm
- net /ROW_A: track 259.7 -> 304.0 mm
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Other:
- board size 300 x 130 mm -> 300 x 132 mm
- board text added: "1 2 3 4 5 6 7 8"
- board text added: "1 2 3 4 5 6 7 8 9 10 11 12 13"

Commit message: Replaced Cherry MX with Gateron LP
Parts:
- SW1, SW10, SW11, SW12, SW13, SW14, SW15, SW16, SW17, SW18, SW19, SW2, SW20, SW21, SW22, SW23, SW24, SW25, SW26, SW27, SW28, SW29, SW3, SW30, SW31, SW32, SW33, SW34, SW35, SW36, SW37, SW38, SW39, SW4, SW40, SW41, SW42, SW43, SW44, SW45, SW46, SW47, SW48, SW49, SW5, SW50, SW51, SW52, SW53, SW54, SW55, SW56, SW57, SW58, SW59, SW6, SW60, SW61, SW62, SW63, SW64, SW65, SW66, SW67, SW68, SW69, SW7, SW70, SW71, SW72, SW8, SW9: footprint PCM_Switch_Keyboard_Cherry_MX:SW_Cherry_MX_PCB_1.00u -> Clueless_Engineer:SW_Gateron_LowProfile_THT
- moved J1 11.7 mm to (57.4, 129.4)
Routing:
- net /ROW_E: track 249.4 -> 281.2 mm
- net /ROW_F: track 261.0 -> 292.8 mm
- net /COL_2: track 403.1 -> 373.8 mm
- net /COL_3: track 384.6 -> 355.5 mm
- net /ROW_G: track 267.9 -> 292.4 mm
- net /ROW_D: track 245.9 -> 265.6 mm
- net /ROW_C: track 248.0 -> 265.9 mm
- net /ROW_H: track 44.7 -> 60.4 mm
- net /ROW_A: track 304.0 -> 292.9 mm
- net /COL_12: track 167.1 -> 178.1 mm
- net /COL_6: track 280.2 -> 269.8 mm
- net /ROW_B: track 263.7 -> 273.2 mm
- net /COL_5: track 323.1 -> 314.1 mm
- net /COL_4: track 344.7 -> 337.2 mm
- net /COL_13: track 155.8 -> 162.0 mm
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Other:
- board size 300 x 132 mm -> 311.7 x 132 mm
