File: Elektronika_K001_DON_Keyboard/Elektronika_K001_DON_Keyboard.kicad_sch (KiCad schematic)
At the start: 74 parts, among them J1 ROWS, J2 COLS, SW1 СБР, SW10 1, SW11 C, SW12 Y, SW13 ⎴, SW14 ↖, SW15 NEW, SW16 2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

Commit message: Replaced Cherry MX with Gateron LP
Parts:
- SW1, SW10, SW11, SW12, SW13, SW14, SW15, SW16, SW17, SW18, SW19, SW2, SW20, SW21, SW22, SW23, SW24, SW25, SW26, SW27, SW28, SW29, SW3, SW30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: footprint PCM_Switch_Keyboard_Cherry_MX:SW_Cherry_MX_PCB_1.00u -> Clueless_Engineer:SW_Gateron_LowProfile_THT
