File: Elektronika_K001_DON_Power/Elektronika_K001_DON_Power.kicad_sch (KiCad schematic)
At the start: 12 parts, among them J1 Power In (+12VDC), J2 Conn_01x05, U1 PSU5, U2 R-78CK5.0-0.5

Commit message: Added fuse on 12V input
Parts:
- added F1: Fuse, Fuse:Fuseholder_Clip-5x20mm_Littelfuse_111_Inline_P20.00x5.00mm_D1.05mm_Horizontal, symbol Device:Fuse
Connections:
- net +12V: now also F1.2; no longer J1.1
- new net +12V_{IN}: F1.1, J1.1
Changed lines of the file:
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@@
-	(wire
-		(pts
-			(xy 76.2 71.12) (xy 97.79 71.12)
-		)
-		(stroke
-			(width 0)
-			(type default)
-		)
-	)
 	(wire
 		(pts
@@
 	(wire
 		(pts
+			(xy 92.71 71.12) (xy 97.79 71.12)
+		)
+		(stroke
+			(width 0)
+			(type default)
+		)
+	)
+	(wire
+		(pts
 			(xy 152.4 87.63) (xy 118.11 87.63)
 		)
@@
 		(pts
 			(xy 124.46 69.85) (xy 124.46 76.2)
+		)
+		(stroke
+			(width 0)
+			(type default)
+		)
+	)
+	(wire
+		(pts
+			(xy 85.09 71.12) (xy 76.2 71.12)
 		)
 		(stroke
@@
 		)
 	)
-	(label "+12V"
-		(at 80.01 71.12 0)
+	(label "+12V_{IN}"
+		(at 77.47 71.12 0)
 		(effects
 			(font
@@
 					(unit 1)
 				)
+			)
+		)
+	)
+	(symbol
+		(lib_id "Device:Fuse")
+		(at 88.9 71.12 90)
+		(unit 1)
+		(exclude_from_sim no)
+		(in_bom yes)
+		(on_board yes)
+		(dnp no)
+		(fields_autoplaced yes)
+		(property "Reference" "F1"
+			(at 88.9 64.77 90)
+			(effects
+				(font
+					(size 1.27 1.27)
+				)
+			)
+		)
+		(property "Value" "Fuse"
+			(at 88.9 67.31 90)
+			(effects
+				(font
+					(size 1.27 1.27)
+				)
+			)
+		)
+		(property "Footprint" "Fuse:Fuseholder_Clip-5x20mm_Littelfuse_111_Inline_P20.00x5.00mm_D1.05mm_Horizontal"
+			(at 88.9 72.898 90)
+			(effects
+				(font
+					(size 1.27 1.27)
+				)
+				(hide yes)
+			)
+		)
+		(property "Datasheet" "~"
+			(at 88.9 71.12 0)
+			(effects
+				(font
+					(size 1.27 1.27)
+				)
+				(hide yes)
+			)
+		)
+		(property "Description" "Fuse"
+			(at 88.9 71.12 0)
+			(effects
+				(font
+					(size 1.27 1.27)
+				)
+				(hide yes)
+			)
+		)
+		(pin "2"
+		)
+		(pin "1"
+		)
+		(instances
+			(project ""
+				(path "/bff640d3-88e6-45d7-956e-e9c03bf1b325"
+					(reference "F1")
+					(unit 1)
+				)
